File: QL_Qsound2.kicad_sch (KiCad schematic)
At the start: 39 parts, among them J1 QL_SLOT_DIN41612_CARD, J2 AudioJack2_Ground_Switch, J3 Conn_02x17_Odd_Even, Q1 2N2369, U1 7805, U2 W27C512, U3 74LS266, U4 6821, U5 LM358, U6 GAL22V10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

Commit message: ADD NOTE
Parts:
- X1, X1B1: value 2Mhz -> 4Mhz
Changed lines of the file:
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@@
 		(title "QSound 2+  for Sinclair QL")
 		(date "2024-11-10")
-		(rev "1")
+		(rev "2")
 		(company "Alvaro Alea Fdz")
 	)
@@
 	(wire
 		(pts
+			(xy 187.96 177.8) (xy 187.96 176.53)
+		)
+		(stroke
+			(width 0)
+			(type default)
+		)
+	)
+	(wire
+		(pts
 			(xy 189.23 213.36) (xy 199.39 213.36)
 		)
@@
 	(wire
 		(pts
+			(xy 187.96 176.53) (xy 191.77 176.53)
+		)
+		(stroke
+			(width 0)
+			(type default)
+		)
+	)
+	(wire
+		(pts
 			(xy 201.93 102.87) (xy 212.09 102.87)
 		)
@@
 	(wire
 		(pts
-			(xy 191.77 162.56) (xy 191.77 170.18)
+			(xy 191.77 162.56) (xy 191.77 176.53)
 		)
 		(stroke
@@
 	(wire
 		(pts
-			(xy 170.18 170.18) (xy 191.77 170.18)
+			(xy 166.37 177.8) (xy 187.96 177.8)
 		)
 		(stroke
@@
 	)
 	(label "E"
-		(at 173.99 170.18 0)
+		(at 170.18 177.8 0)
 		(fields_autoplaced yes)
 		(effects
@@
 		(on_board yes)
 		(dnp no)
-		(fields_autoplaced yes)
 		(property "Reference" "X1"
-			(at 179.07 146.2121 0)
+			(at 177.8 146.0814 0)
 			(effects
 				(font
@@
 			)
 		)
-		(property "Value" "2Mhz"
+		(property "Value" "4Mhz"
 			(at 181.61 148.7521 0)
 			(do_not_autoplace yes)
@@
 			)
 		)
-		(property "Value" "2Mhz"
+		(property "Value" "4Mhz"
 			(at 203.2 148.7521 0)
 			(do_not_autoplace yes)

Commit message: new clock oscilators
Parts:
- removed X1: 4Mhz, Oscillator:Oscillator_DIP-8, symbol Oscillator:CXO_DIP8
- added U10: 74HC74, Package_DIP:DIP-14_W7.62mm_LongPads, symbol 74xx:74HC74
- added X3: 3Mhz, Oscillator:Oscillator_SMD_Abracon_ASV-4Pin_7.0x5.1mm, symbol Oscillator:DFA-S2
- X4: renamed from X1B1; footprint Oscillator:Oscillator_SMD_Abracon_ASE-4Pin_3.2x2.5mm_HandSoldering -> Oscillator:Oscillator_SMD_Abracon_ASV-4Pin_7.0x5.1mm
Connections:
- net E: no longer JP1.1 (A)
- net GND: now also U10.7 (GND), X3.2 (GND)
- net VCC: now also U10.1 (~{R}), U10.10 (~{S}), U10.13 (~{R}), U10.14 (VCC), U10.4 (~{S}), X3.4 (V+); no longer X4.1 (Vctrl)
- net at JP1.3 (B): now also U10.5 (Q); no longer X4.3 (OUT)
- new net: U10.2 (D), U10.6 (~{Q})
- new net: U10.3 (C), X3.3 (OUT)
- new net: JP1.1 (A), X4.3 (OUT)
- no-connect marks 47 -> 49
Other:
- moved on the sheet: U8, X4
